File: Contact-Monitor-Board.kicad_pcb (KiCad board)
At the start: 2 copper layers, 100 x 100 mm, 82 parts, among them J1 Screw_Terminal_01x02, J10 Screw_Terminal_01x02, J11 Screw_Terminal_01x02, J12 Screw_Terminal_01x02, J13 Screw_Terminal_01x02, J14 Screw_Terminal_01x02, J15 Screw_Terminal_01x02, J16 Screw_Terminal_01x02, J2 Screw_Terminal_01x02, J3 Screw_Terminal_01x02, J4 Screw_Terminal_01x02, J5 Screw_Terminal_01x02, J6 Screw_Terminal_01x02, J7 Screw_Terminal_01x02, J8 Screw_Terminal_01x02, J9 Screw_Terminal_01x02, Q1 2N7002, Q10 2N7002, Q11 2N7002, Q12 2N7002, Q13 2N7002, Q14 2N7002, Q15 2N7002, Q16 2N7002, Q2 2N7002, Q3 2N7002, Q4 2N7002, Q5 2N7002, Q6 2N7002, Q7 2N7002, Q8 2N7002, Q9 2N7002, SW1 SW_Nidec_CAS-120A1, U1 74HC4017D, U2 TLC555CD, U3 TPS61222DCK

Commit message: バージョン表記修正
Other:
- board text added: "CONTACT MONITOR BOARD V1.1"
- board text removed: "CONTACT MONITOR BOARD V1.0"
Changed lines of the file:
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@@
 		(title "Contact Monitor Board")
 		(date "2026-08-04")
-		(rev "1.0")
+		(rev "1.1")
 		(company "Satoru Yamaguchi")
 		(comment 1 "Copyright (c) 2026 Satoru Yamaguchi")
@@
 		)
 	)
-	(gr_text "CONTACT MONITOR BOARD\nV1.0"
+	(gr_text "CONTACT MONITOR BOARD\nV1.1"
 		(at 156.614 40.798 0)
 		(layer "F.SilkS")
