File: Contact-Monitor-Board.kicad_pcb (KiCad board)
At the start: 2 copper layers, 100 x 100 mm, 83 parts, among them J1 JST VH 02, J10 JST VH 02, J11 JST VH 02, J12 JST VH 02, J13 JST VH 02, J14 JST VH 02, J15 JST VH 02, J16 JST VH 02, J17 header 4, J2 JST VH 02, J3 JST VH 02, J4 JST VH 02, J5 JST VH 02, J6 JST VH 02, J7 JST VH 02, J8 JST VH 02, J9 JST VH 02, Q1 2N7002, Q10 2N7002, Q11 2N7002, Q12 2N7002, Q13 2N7002, Q14 2N7002, Q15 2N7002, Q16 2N7002, Q2 2N7002, Q3 2N7002, Q4 2N7002, Q5 2N7002, Q6 2N7002, Q7 2N7002, Q8 2N7002, Q9 2N7002, SW1 KH-SS12D01-G3-5.0, U1 74HC4017D, U2 TLC555CD, U3 TPS61222DCK

Commit message: 運転LED輝度調整 R1 470 -> 1k
Parts:
- R1: value 470 -> 1.0k
Changed lines of the file:
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@@
 			)
 		)
-		(property "Value" "470"
+		(property "Value" "1.0k"
 			(at 0 1.43 0)
 			(layer "F.Fab")
@@
 			)
 		)
-		(property "LCSC" "C23179"
+		(property "LCSC" "C21190"
 			(at 0 0 0)
 			(layer "F.SilkS")
